Commit message: small modifications

File: src/mybot/urdf/lidar.xacro (robot description, xacro)
@@ -8,4 +8,9 @@
     </joint>
     <link name="lidar">
+        <inertial>
+          <origin xyz="0.0 0.0 0.0" rpy="0.0 0.0 0.0"/>
+          <mass value="0.25"/>
+          <inertia ixx="1e-6" ixy="0.0" ixz="0.0" iyy="1e-6" iyz="0.0" izz="1e-6"/>
+        </inertial>
         <visual>
             <geometry>
@@ -31,10 +36,10 @@
                     <resolution>1</resolution>
                     <min_angle>-3.14159</min_angle>
-                    <max_angle>3.14159*2</max_angle>
+                    <max_angle>3.14159</max_angle>
                 </horizontal>
                 </scan>
                 <range>
                     <min>0.10</min>
-                    <max>8.0</max>
+                    <max>30.0</max>
                     <resolution>0.01</resolution>
                 </range>

File: src/mybot/urdf/skid_steering.xacro (robot description, xacro)
@@ -12,5 +12,5 @@
             <wheelDiameter>0.4</wheelDiameter>
             <robotBaseFrame>robot_footprint</robotBaseFrame>
-            <torque>30</torque>
+            <torque>50</torque>
             <topicName>cmd_vel</topicName>
             <broadcastTF>true</broadcastTF>
